File: Hardware/control v1.brd (EAGLE design)
At the start: 100 x 100 mm, 51 parts, among them T1 2N3904, T2 2N3904

Commit message: correct values
Parts:
- removed R2, R4, R6, R8: 68R, resistor-mod:0207/7
- POT1, POT2, POT3, POT4, POT5, POT6, POT7, POT8: value (none) -> 10K
- R1, R3, R5, R7: value 68R -> 34,8R
- moved R5 11.4 mm to (53.3, 38.7)
- moved R7 11.4 mm to (71.1, 38.7)
- moved R3 10.8 mm to (35.6, 38.7)
- moved POT1 1.00 mm to (14.0, 87.0)
- moved POT2 1.00 mm to (38.0, 87.0)
- moved POT4 1.00 mm to (86.0, 87.0)
- moved POT5 1.00 mm to (14.0, 62.0)
- moved POT6 1.00 mm to (38.0, 62.0)
- moved POT8 1.00 mm to (86.0, 62.0)
- moved C1 0.63 mm to (94.6, 84.5)
- renumbered JP3 to JP3-AUDIO
Connections:
- net GND: now also A-IN1.P$2_SWITCH; no longer R4.2, R6.2, R8.2
- net L1: no longer R2.1
- net N$3: no longer R4.1
- net N$4: no longer R6.1
- net N$5: no longer R2.2
- net N$6: no longer R8.1
- net POT5: now also JP-POT.8; no longer JP-POT.10
- net POT6: now also JP-POT.10; no longer JP-POT.9
- net POT7: now also JP-POT.9; no longer JP-POT.8
Routing:
- net POT2: track 51.6 -> 37.9 mm
- net N$4: track 11.5 -> 5.69 mm
- net POT7: track 71.6 -> 77.4 mm
- net N$6: track 11.5 -> 5.91 mm
- net N$3: track 10.8 -> 5.47 mm
- net POT6: track 55.5 -> 51.2 mm
- net B2: track 77.1 -> 80.4 mm
- net N$5: track 6.58 -> 3.40 mm
- net +3V3: track 175.4 -> 172.8 mm
- net B3: track 57.7 -> 59.9 mm
- net L1: track 90.0 -> 87.8 mm
- net L2: track 77.3 -> 75.8 mm
- net POT4: track 85.9 -> 87.0 mm
- net B4: track 35.1 -> 34.0 mm
- net POT5: track 20.1 -> 21.2 mm
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Other:
- board text added: "1"
- board text added: "2"
- board text added: "3"
- board text added: "4"
- board text added: "5"
- board text added: "6"
- board text added: "7"
- board text added: "8"
- board text added: "B1"
- board text added: "B2"
- board text added: "B3"
- board text added: "B4"
- board text added: "CC-BY-SA-NC"
- board text added: "CONTROL"
- board text added: "EUXOLOTI"
- board text added: "G1"
- board text added: "G2"
- board text added: "I"
- board text added: "L1"
- board text added: "L2"
- board text added: "L3"
- board text added: "L4"
- board text added: "O"
- board text added: "PCB VERSION 1.00"
- board text added: "by Paul 2015"
- board text added: "www.irieelectronics.de"
