File: Hardware/control v1.sch (EAGLE design)
At the start: 51 parts, among them T1 2N3904, T2 2N3904

Commit message: correct values
Parts:
- removed R2, R4, R6, R8: 68R, resistor-mod:R-EU_0207/7
- POT1, POT2, POT3, POT4, POT5, POT6, POT7, POT8: value (none) -> 10K
- R1, R3, R5, R7: value 68R -> 34,8R
- renumbered JP3 to JP3-AUDIO
Connections:
- net GND: now also A-IN1.SWITCH; no longer R4.2, R6.2, R8.2
- net L1: no longer R2.1
- net N$3: no longer R4.1
- net N$4: no longer R6.1
- net N$5: no longer R2.2
- net N$6: no longer R8.1
- net POT5: now also JP-POT.8; no longer JP-POT.10
- net POT6: now also JP-POT.10; no longer JP-POT.9
- net POT7: now also JP-POT.9; no longer JP-POT.8
Changed lines of the file:
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@@
 </classes>
 <parts>
-<part name="POT1" library="MusicThingModular" deviceset="9MM_SNAP-IN_POT" device="_"/>
-<part name="POT2" library="MusicThingModular" deviceset="9MM_SNAP-IN_POT" device="_"/>
-<part name="POT3" library="MusicThingModular" deviceset="9MM_SNAP-IN_POT" device="_"/>
-<part name="POT4" library="MusicThingModular" deviceset="9MM_SNAP-IN_POT" device="_"/>
-<part name="POT5" library="MusicThingModular" deviceset="9MM_SNAP-IN_POT" device="_"/>
-<part name="POT6" library="MusicThingModular" deviceset="9MM_SNAP-IN_POT" device="_"/>
-<part name="POT7" library="MusicThingModular" deviceset="9MM_SNAP-IN_POT" device="_"/>
-<part name="POT8" library="MusicThingModular" deviceset="9MM_SNAP-IN_POT" device="_"/>
+<part name="POT1" library="MusicThingModular" deviceset="9MM_SNAP-IN_POT" device="_" value="10K"/>
+<part name="POT2" library="MusicThingModular" deviceset="9MM_SNAP-IN_POT" device="_" value="10K"/>
+<part name="POT3" library="MusicThingModular" deviceset="9MM_SNAP-IN_POT" device="_" value="10K"/>
+<part name="POT4" library="MusicThingModular" deviceset="9MM_SNAP-IN_POT" device="_" value="10K"/>
+<part name="POT5" library="MusicThingModular" deviceset="9MM_SNAP-IN_POT" device="_" value="10K"/>
+<part name="POT6" library="MusicThingModular" deviceset="9MM_SNAP-IN_POT" device="_" value="10K"/>
+<part name="POT7" library="MusicThingModular" deviceset="9MM_SNAP-IN_POT" device="_" value="10K"/>
+<part name="POT8" library="MusicThingModular" deviceset="9MM_SNAP-IN_POT" device="_" value="10K"/>
 <part name="JP-POT" library="pinhead 2" deviceset="PINHD-1X10" device="_2.54"/>
 <part name="B1" library="og-switch" deviceset="LP4OA1PBCTG" device=""/>
@@
 <part name="GND20" library="supply1" deviceset="GND" device=""/>
 <part name="JP3-CV" library="pinhead" deviceset="PINHD-1X8" device=""/>
-<part name="R1" library="resistor-mod" deviceset="R-EU_" device="0207/7" value="68R"/>
-<part name="R2" library="resistor-mod" deviceset="R-EU_" device="0207/7" value="68R"/>
-<part name="R3" library="resistor-mod" deviceset="R-EU_" device="0207/7" value="68R"/>
-<part name="R4" library="resistor-mod" deviceset="R-EU_" device="0207/7" value="68R"/>
-<part name="R5" library="resistor-mod" deviceset="R-EU_" device="0207/7" value="68R"/>
-<part name="R6" library="resistor-mod" deviceset="R-EU_" device="0207/7" value="68R"/>
-<part name="R7" library="resistor-mod" deviceset="R-EU_" device="0207/7" value="68R"/>
-<part name="R8" library="resistor-mod" deviceset="R-EU_" device="0207/7" value="68R"/>
-<part name="JP3" library="pinhead" deviceset="PINHD-1X4" device=""/>
+<part name="R1" library="resistor-mod" deviceset="R-EU_" device="0207/7" value="34,8R"/>
+<part name="R3" library="resistor-mod" deviceset="R-EU_" device="0207/7" value="34,8R"/>
+<part name="R5" library="resistor-mod" deviceset="R-EU_" device="0207/7" value="34,8R"/>
+<part name="R7" library="resistor-mod" deviceset="R-EU_" device="0207/7" value="34,8R"/>
+<part name="JP3-AUDIO" library="pinhead" deviceset="PINHD-1X4" device=""/>
 <part name="JP1" library="pinhead" deviceset="PINHD-1X30" device=""/>
 <part name="GND21" library="supply1" deviceset="GND" device=""/>
@@
 </segment>
 <segment>
+<pinref part="JP-POT" gate="A" pin="8"/>
+<wire x1="93.98" y1="76.2" x2="88.9" y2="76.2" width="0.1524" layer="91"/>
+<label x="88.9" y="76.2" size="1.016" layer="95" rot="R180" xref="yes"/>
+</segment>
+</net>
+<net name="POT6" class="0">
+<segment>
+<pinref part="POT6" gate="G$1" pin="S"/>
+<wire x1="35.56" y1="63.5" x2="38.1" y2="63.5" width="0.1524" layer="91"/>
+<label x="38.1" y="63.5" size="1.778" layer="95" xref="yes"/>
+</segment>
+<segment>
 <pinref part="JP-POT" gate="A" pin="10"/>
 <wire x1="93.98" y1="71.12" x2="88.9" y2="71.12" width="0.1524" layer="91"/>
@@
 </segment>
 </net>
-<net name="POT6" class="0">
-<segment>
-<pinref part="POT6" gate="G$1" pin="S"/>
-<wire x1="35.56" y1="63.5" x2="38.1" y2="63.5" width="0.1524" layer="91"/>
-<label x="38.1" y="63.5" size="1.778" layer="95" xref="yes"/>
+<net name="POT7" class="0">
+<segment>
+<pinref part="POT7" gate="G$1" pin="S"/>
+<wire x1="35.56" y1="38.1" x2="38.1" y2="38.1" width="0.1524" layer="91"/>
+<label x="38.1" y="38.1" size="1.778" layer="95" xref="yes"/>
 </segment>
 <segment>
@@
 <wire x1="93.98" y1="73.66" x2="88.9" y2="73.66" width="0.1524" layer="91"/>
 <label x="88.9" y="73.66" size="1.016" layer="95" rot="R180" xref="yes"/>
-</segment>
-</net>
-<net name="POT7" class="0">
-<segment>
-<pinref part="POT7" gate="G$1" pin="S"/>
-<wire x1="35.56" y1="38.1" x2="38.1" y2="38.1" width="0.1524" layer="91"/>
-<label x="38.1" y="38.1" size="1.778" layer="95" xref="yes"/>
-</segment>
-<segment>
-<pinref part="JP-POT" gate="A" pin="8"/>
-<wire x1="93.98" y1="76.2" x2="88.9" y2="76.2" width="0.1524" layer="91"/>
-<label x="88.9" y="76.2" size="1.016" layer="95" rot="R180" xref="yes"/>
 </segment>
 </net>
@@
 <instance part="GND12" gate="1" x="162.56" y="35.56"/>
 <instance part="R1" gate="G$1" x="-12.7" y="68.58"/>
-<instance part="R2" gate="G$1" x="-12.7" y="76.2"/>
 <instance part="R3" gate="G$1" x="58.42" y="71.12"/>
-<instance part="R4" gate="G$1" x="58.42" y="76.2"/>
 <instance part="R5" gate="G$1" x="111.76" y="71.12"/>
-<instance part="R6" gate="G$1" x="111.76" y="76.2"/>
 <instance part="R7" gate="G$1" x="157.48" y="71.12"/>
-<instance part="R8" gate="G$1" x="157.48" y="76.2"/>
 </instances>
 <busses>
@@
 <junction x="63.5" y="43.18"/>
 <pinref part="R3" gate="G$1" pin="2"/>
-<pinref part="R4" gate="G$1" pin="2"/>
-<wire x1="63.5" y1="76.2" x2="63.5" y2="71.12" width="0.1524" layer="91"/>
-<junction x="63.5" y="71.12"/>
 </segment>
 <segment>
@@
 <junction x="116.84" y="43.18"/>
 <pinref part="R5" gate="G$1" pin="2"/>
-<pinref part="R6" gate="G$1" pin="2"/>
-<wire x1="116.84" y1="76.2" x2="116.84" y2="71.12" width="0.1524" layer="91"/>
-<junction x="116.84" y="71.12"/>
 </segment>
 <segment>
@@
 <junction x="162.56" y="43.18"/>
 <pinref part="R7" gate="G$1" pin="2"/>
-<pinref part="R8" gate="G$1" pin="2"/>
-<wire x1="162.56" y1="76.2" x2="162.56" y2="71.12" width="0.1524" layer="91"/>
-<junction x="162.56" y="71.12"/>
 </segment>
 </net>
 <net name="N$5" class="0">
 <segment>
-<pinref part="R2" gate="G$1" pin="2"/>
 <pinref part="R1" gate="G$1" pin="2"/>
-<wire x1="-7.62" y1="76.2" x2="-7.62" y2="68.58" width="0.1524" layer="91"/>
 <pinref part="B1" gate="G$1" pin="L1"/>
 <wire x1="-7.62" y1="68.58" x2="-5.08" y2="68.58" width="0.1524" layer="91"/>
-<junction x="-7.62" y="68.58"/>
 </segment>
 </net>
 <net name="L1" class="0">
 <segment>
-<pinref part="R2" gate="G$1" pin="1"/>
 <pinref part="R1" gate="G$1" pin="1"/>
-<wire x1="-17.78" y1="76.2" x2="-17.78" y2="68.58" width="0.1524" layer="91"/>
 <wire x1="-17.78" y1="68.58" x2="-20.32" y2="68.58" width="0.1524" layer="91"/>
-<junction x="-17.78" y="68.58"/>
 <label x="-20.32" y="68.58" size="1.778" layer="95" rot="R180" xref="yes"/>
 </segment>
@@
 <pinref part="B2" gate="G$1" pin="L2"/>
 <pinref part="R3" gate="G$1" pin="1"/>
-<pinref part="R4" gate="G$1" pin="1"/>
-<wire x1="53.34" y1="76.2" x2="53.34" y2="71.12" width="0.1524" layer="91"/>
-<junction x="53.34" y="71.12"/>
 </segment>
 </net>
@@
 <pinref part="B3" gate="G$1" pin="L2"/>
 <pinref part="R5" gate="G$1" pin="1"/>
-<pinref part="R6" gate="G$1" pin="1"/>
-<wire x1="106.68" y1="76.2" x2="106.68" y2="71.12" width="0.1524" layer="91"/>
-<junction x="106.68" y="71.12"/>
 </segment>
 </net>
@@
 <pinref part="B4" gate="G$1" pin="L2"/>
 <pinref part="R7" gate="G$1" pin="1"/>
-<pinref part="R8" gate="G$1" pin="1"/>
-<wire x1="152.4" y1="76.2" x2="152.4" y2="71.12" width="0.1524" layer="91"/>
-<junction x="152.4" y="71.12"/>
 </segment>
 </net>
@@
 </plain>
 <instances>
-<instance part="JP3" gate="A" x="53.34" y="27.94"/>
+<instance part="JP3-AUDIO" gate="A" x="53.34" y="27.94"/>
 <instance part="A-IN1" gate="G$1" x="-5.08" y="73.66" rot="MR0"/>
 <instance part="A-OUT2" gate="G$1" x="50.8" y="55.88"/>
@@
 </segment>
 <segment>
-<pinref part="JP3" gate="A" pin="1"/>
+<pinref part="JP3-AUDIO" gate="A" pin="1"/>
 <wire x1="50.8" y1="33.02" x2="45.72" y2="33.02" width="0.1524" layer="91"/>
 <label x="45.72" y="33.02" size="1.016" layer="95" rot="R180" xref="yes"/>
@@
 </segment>
 <segment>
-<pinref part="JP3" gate="A" pin="4"/>
+<pinref part="JP3-AUDIO" gate="A" pin="4"/>
 <wire x1="50.8" y1="25.4" x2="45.72" y2="25.4" width="0.1524" layer="91"/>
 <label x="45.72" y="25.4" size="1.016" layer="95" rot="R180" xref="yes"/>
@@
 </segment>
 <segment>
-<pinref part="JP3" gate="A" pin="2"/>
+<pinref part="JP3-AUDIO" gate="A" pin="2"/>
 <wire x1="50.8" y1="30.48" x2="45.72" y2="30.48" width="0.1524" layer="91"/>
 <label x="45.72" y="30.48" size="1.016" layer="95" rot="R180" xref="yes"/>
@@
 </segment>
 <segment>
-<pinref part="JP3" gate="A" pin="3"/>
+<pinref part="JP3-AUDIO" gate="A" pin="3"/>
 <wire x1="50.8" y1="27.94" x2="45.72" y2="27.94" width="0.1524" layer="91"/>
 <label x="45.72" y="27.94" size="1.016" layer="95" rot="R180" xref="yes"/>
@@
 <pinref part="A-IN1" gate="G$1" pin="SLEEVE"/>
 <pinref part="GND15" gate="1" pin="GND"/>
-</segment>
-</net>
+<pinref part="A-IN1" gate="G$1" pin="SWITCH"/>
+<wire x1="0" y1="73.66" x2="0" y2="71.12" width="0.1524" layer="91"/>
+<junction x="0" y="71.12"/>
+</segment>
+</net>
