File: Hardware/core v1.brd (EAGLE design)
At the start: 100 x 100 mm, 90 parts, among them IC1 7805, IC2 TL074P, IC3 MCP6004, IC4 MCP6004

Commit message: correct values
Parts:
- C22, C24: value (none) -> 10uF
- R13, R34: value 60k -> 33K
- R19: value 60k -> 66,5K
- R25, R26, R28, R35, R8: value 30k -> 33K
- moved JP1-AU_FROM_AXO 1.27 mm to (66.7, 85.7)
- moved C7 0.64 mm to (78.7, 79.4)
- moved L2 0.64 mm to (24.8, 94.6)
- turned C1 to 270 degrees
- turned C2 to 270 degrees
Routing:
- net N$14: track 11.0 -> 12.3 mm
- net N$1: track 2.54 -> 3.18 mm
- net VEE: track 62.8 -> 62.2 mm
- net VDD: track 146.3 -> 145.8 mm
Other:
- board text added: "0"
- board text added: "1"
- board text added: "2"
- board text added: "3"
- board text added: "4"
- board text added: "5"
- board text added: "6"
- board text added: "7"
- board text added: "ch:"
- board text added: "in1"
- board text added: "in2"
- board text added: "out1"
- board text added: "out2"
