File: Hardware/euxoloti core rev2.brd (EAGLE design)
At the start: 100 x 100 mm, 90 parts, among them IC1 7805, IC2 TL074P, IC3 MCP6004, IC4 MCP6004

Commit message: update REV 2
Parts:
- removed R41: 47K, resistor-mod:0207/7
- R14, R16: value 3,3K -> 15K
- R2, R6: value 3,3K -> 1K
- moved C4 9.92 mm to (38.7, 95.2), flipped to the bottom, turned to 90 degrees
- moved R40 5.24 mm to (48.3, 83.2)
- moved IC1 3.81 mm to (36.2, 87.6)
- moved D3 3.59 mm to (54.6, 47.0), turned to 0 degrees
- moved D4 2.69 mm to (50.2, 86.4)
- moved C25 2.54 mm to (67.3, 94.0)
- moved JP1 1.80 mm to (52.7, 71.8), turned to 0 degrees
- moved JP1-AU_FROM_AXO 1.27 mm to (65.4, 85.7)
- moved L3 0.90 mm to (50.2, 90.8)
- moved C3 0.63 mm to (45.1, 95.2)
- moved R3 0.63 mm to (76.2, 90.8)
- turned C24 to 270 degrees
Connections:
- new net LIN-: AXOLOTICORE.LIN-, C22.+
- new net RIN-: AXOLOTICORE.RIN-, C24.+
- net AREF_-10: now also D3.-; no longer D3.2
- net GND: now also AXOLOTICORE.GND4, AXOLOTICORE.GND5, D3.+; no longer D3.1, R41.2
- net LIN+: no longer C22.+
- net RIN+: no longer C24.+
- net VBUS: no longer R41.1
Routing:
- net LIN-: track 0.00 -> 18.9 mm
- net LIN+: track 17.9 -> 0.00 mm
- net RIN+: track 9.58 -> 0.00 mm
- net AREF_-10: track 168.1 -> 163.9 mm
- net VCC: track 81.9 -> 78.2 mm
- net RIN-: track 0.00 -> 2.92 mm
- net N$19: track 71.1 -> 72.6 mm
- net N$14: track 12.3 -> 13.5 mm
- net N$13: track 20.3 -> 21.5 mm
- net CM: track 82.8 -> 83.8 mm
- net +5V: track 13.3 -> 14.2 mm
- net N$16: track 8.00 -> 8.89 mm
- net +3V3: track 97.9 -> 97.2 mm
- net N$4: track 7.62 -> 6.98 mm
- net +5V_RAW: track 12.7 -> 13.3 mm
