File: Hardware/euxoloti core rev2.sch (EAGLE design)
At the start: 89 parts, among them IC1 7805, IC2 TL074P, IC3 MCP6004, IC4 MCP6004

Commit message: update REV 2
Parts:
- removed R41: 47K, resistor-mod:R-EU_0207/7
- R14, R16: value 3,3K -> 15K
- R2, R6: value 3,3K -> 1K
Connections:
- new net LIN-: AXOLOTICOREG$1.LIN-, C22.+
- new net RIN-: AXOLOTICOREG$1.RIN-, C24.+
- net AREF_-10: now also D3.-; no longer D3.A
- net GND: now also AXOLOTICOREG$1.GND4, AXOLOTICOREG$1.GND5, D3.+; no longer D3.C, R41.2
- net LIN+: no longer C22.+
- net RIN+: no longer C24.+
- net VBUS: no longer R41.1
Other:
- note removed: "in: 10Vpp"
- note removed: "out: 1,5Vpp"
Changed lines of the file:
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@@
 <part name="GND18" library="SparkFun" deviceset="GND" device=""/>
 <part name="R1" library="resistor-mod" deviceset="R-EU_" device="0207/10" value="22K"/>
-<part name="R2" library="resistor-mod" deviceset="R-EU_" device="0207/12" value="3,3K"/>
+<part name="R2" library="resistor-mod" deviceset="R-EU_" device="0207/12" value="1K"/>
 <part name="R3" library="resistor-mod" deviceset="R-TRIMM" device="3296P" value="5K"/>
 <part name="R4" library="resistor-mod" deviceset="R-EU_" device="0207/7" value="1K"/>
 <part name="R5" library="resistor-mod" deviceset="R-EU_" device="0207/7" value="22K"/>
-<part name="R6" library="resistor-mod" deviceset="R-EU_" device="0207/7" value="3,3K"/>
+<part name="R6" library="resistor-mod" deviceset="R-EU_" device="0207/7" value="1K"/>
 <part name="R11" library="resistor-mod" deviceset="R-TRIMM" device="3296P" value="5K"/>
 <part name="R12" library="resistor-mod" deviceset="R-EU_" device="0207/10" value="1K"/>
 <part name="GND33" library="SparkFun" deviceset="GND" device=""/>
 <part name="JP1-AU_FROM_AXO" library="pinhead" deviceset="PINHD-1X2" device="/90"/>
-<part name="R14" library="resistor-mod" deviceset="R-EU_" device="0207/7" value="3,3K"/>
+<part name="R14" library="resistor-mod" deviceset="R-EU_" device="0207/7" value="15K"/>
 <part name="R15" library="resistor-mod" deviceset="R-EU_" device="0207/7" value="22K"/>
-<part name="R16" library="resistor-mod" deviceset="R-EU_" device="0207/7" value="3,3K"/>
+<part name="R16" library="resistor-mod" deviceset="R-EU_" device="0207/7" value="15K"/>
 <part name="R31" library="resistor-mod" deviceset="R-EU_" device="0207/7" value="22K"/>
 <part name="+3V13" library="supply1" deviceset="+3V3" device=""/>
@@
 <part name="GND10" library="supply1" deviceset="GND" device=""/>
 <part name="R40" library="resistor-mod" deviceset="R-EU_" device="0207/7" value="47K"/>
-<part name="R41" library="resistor-mod" deviceset="R-EU_" device="0207/7" value="47K"/>
 <part name="GND12" library="SparkFun" deviceset="GND" device=""/>
 <part name="P+5" library="SparkFun" deviceset="VCC" device=""/>
@@
 <text x="-48.26" y="-63.5" size="1.778" layer="97">-5.0 to 5.0</text>
 <text x="-127" y="-63.5" size="1.778" layer="97">0.0 to 5.0</text>
-<text x="46.228" y="54.102" size="1.778" layer="104">out: 1,5Vpp</text>
-<text x="-16.002" y="42.164" size="1.778" layer="104">in: 10Vpp</text>
 <text x="193.04" y="-134.62" size="2.54" layer="95">1</text>
 <text x="101.6" y="-111.76" size="2.54" layer="95">Paul 2015</text>
@@
 </segment>
 </net>
-<net name="LIN+" class="0">
-<segment>
-<wire x1="66.04" y1="50.8" x2="71.12" y2="50.8" width="0.1524" layer="91"/>
-<pinref part="C22" gate="G$1" pin="+"/>
-<label x="71.12" y="50.8" size="1.778" layer="95" xref="yes"/>
-</segment>
-</net>
 <net name="N$21" class="0">
 <segment>
@@
 <wire x1="129.54" y1="40.64" x2="127" y2="40.64" width="0.1524" layer="91"/>
 <junction x="127" y="40.64"/>
-</segment>
-</net>
-<net name="RIN+" class="0">
-<segment>
-<wire x1="147.32" y1="50.8" x2="152.4" y2="50.8" width="0.1524" layer="91"/>
-<pinref part="C24" gate="G$1" pin="+"/>
-<label x="152.4" y="50.8" size="1.778" layer="95" xref="yes"/>
 </segment>
 </net>
@@
 <wire x1="106.68" y1="38.1" x2="109.22" y2="38.1" width="0.1524" layer="91"/>
 <label x="106.68" y="33.02" size="1.778" layer="95" rot="R270"/>
+</segment>
+</net>
+<net name="LIN-" class="0">
+<segment>
+<wire x1="66.04" y1="50.8" x2="71.12" y2="50.8" width="0.1524" layer="91"/>
+<pinref part="C22" gate="G$1" pin="+"/>
+<label x="71.12" y="50.8" size="1.778" layer="95" xref="yes"/>
+</segment>
+</net>
+<net name="RIN-" class="0">
+<segment>
+<wire x1="147.32" y1="50.8" x2="152.4" y2="50.8" width="0.1524" layer="91"/>
+<pinref part="C24" gate="G$1" pin="+"/>
+<label x="152.4" y="50.8" size="1.778" layer="95" xref="yes"/>
 </segment>
 </net>
@@
 <wire x1="40.64" y1="134.62" x2="53.34" y2="134.62" width="0.1524" layer="91"/>
 <junction x="53.34" y="134.62"/>
+<pinref part="AXOLOTICORE" gate="G$1" pin="GND4"/>
+<wire x1="76.2" y1="124.46" x2="68.58" y2="124.46" width="0.1524" layer="91"/>
+<wire x1="68.58" y1="124.46" x2="68.58" y2="134.62" width="0.1524" layer="91"/>
+<pinref part="AXOLOTICORE" gate="G$1" pin="GND5"/>
+<wire x1="76.2" y1="121.92" x2="68.58" y2="121.92" width="0.1524" layer="91"/>
+<wire x1="68.58" y1="121.92" x2="68.58" y2="124.46" width="0.1524" layer="91"/>
+<junction x="68.58" y="124.46"/>
 </segment>
 <segment>
@@
 <wire x1="149.86" y1="198.12" x2="144.78" y2="198.12" width="0.1524" layer="91"/>
 <label x="144.78" y="198.12" size="1.016" layer="95" rot="R180" xref="yes"/>
+</segment>
+</net>
+<net name="LIN-" class="0">
+<segment>
+<pinref part="AXOLOTICORE" gate="G$1" pin="LIN-"/>
+<wire x1="76.2" y1="116.84" x2="71.12" y2="116.84" width="0.1524" layer="91"/>
+<label x="71.12" y="116.84" size="1.778" layer="95" rot="R180" xref="yes"/>
+</segment>
+</net>
+<net name="RIN-" class="0">
+<segment>
+<pinref part="AXOLOTICORE" gate="G$1" pin="RIN-"/>
+<wire x1="76.2" y1="111.76" x2="71.12" y2="111.76" width="0.1524" layer="91"/>
+<label x="71.12" y="111.76" size="1.778" layer="95" rot="R180" xref="yes"/>
 </segment>
 </net>
@@
 <instance part="TP-10V" gate="G$1" x="106.68" y="0"/>
 <instance part="R40" gate="G$1" x="15.24" y="71.12" rot="R270"/>
-<instance part="R41" gate="G$1" x="25.4" y="55.88" rot="R270"/>
 <instance part="GND12" gate="1" x="25.4" y="45.72"/>
 <instance part="P+5" gate="1" x="15.24" y="78.74"/>
@@
 <pinref part="C16" gate="G$1" pin="2"/>
 <pinref part="GND69" gate="1" pin="GND"/>
-<pinref part="D3" gate="G$1" pin="C"/>
+<pinref part="D3" gate="G$1" pin="+"/>
 </segment>
 <segment>
@@
 </segment>
 <segment>
-<pinref part="R41" gate="G$1" pin="2"/>
 <pinref part="GND12" gate="1" pin="GND"/>
 <wire x1="25.4" y1="48.26" x2="25.4" y2="50.8" width="0.1524" layer="91"/>
@@
 <pinref part="R30" gate="G$1" pin="2"/>
 <pinref part="C16" gate="G$1" pin="1"/>
-<pinref part="D3" gate="G$1" pin="A"/>
+<pinref part="D3" gate="G$1" pin="-"/>
 <wire x1="91.44" y1="-10.16" x2="91.44" y2="-7.62" width="0.1524" layer="91"/>
 <wire x1="96.52" y1="-7.62" x2="96.52" y2="0" width="0.1524" layer="91"/>
@@
 <pinref part="R40" gate="G$1" pin="2"/>
 <wire x1="15.24" y1="66.04" x2="15.24" y2="60.96" width="0.1524" layer="91"/>
-<pinref part="R41" gate="G$1" pin="1"/>
-<wire x1="15.24" y1="60.96" x2="25.4" y2="60.96" width="0.1524" layer="91"/>
 <pinref part="C25" gate="G$1" pin="1"/>
 <wire x1="15.24" y1="60.96" x2="15.24" y2="58.42" width="0.1524" layer="91"/>
 <junction x="15.24" y="60.96"/>
 <pinref part="D4" gate="1" pin="C"/>
-<wire x1="25.4" y1="60.96" x2="35.56" y2="60.96" width="0.1524" layer="91"/>
-<junction x="25.4" y="60.96"/>
+<wire x1="15.24" y1="60.96" x2="35.56" y2="60.96" width="0.1524" layer="91"/>
 <wire x1="35.56" y1="60.96" x2="48.26" y2="60.96" width="0.1524" layer="91"/>
 <junction x="35.56" y="60.96"/>
