File: Hardware/gat8 rev 1.sch (EAGLE design)
At the start: 69 parts, among them IC1 74LS595N, IC2 LP2950ACZ-3.3, T1 2N3904, T2 2N3904, T3 2N3904, T4 2N3904, T5 2N3904, T6 2N3904, T7 2N3904, T8 2N3904

Commit message: update
Parts:
- added SLV: (no value), resistor-mod:R-EU_R0805
- added U$9: LABEL_COMPLETE, labels links:LABEL_COMPLETE
- C4: value 2,2uF -> 47uF
- C5: value 1uF -> 47uF
- C6: value (none) -> 100nF
- D1: value 1N4004 -> 1N4001
- IC2: value LP2950ACZ-3.3 -> LM117-3.3V; device v-reg:LP2950ACZ-3.3 -> v-reg mod:LM117-SOT223
- R25, R26, R27, R28, R29, R30, R31, R32: value 1K -> 2,2K
- renumbered D2 to D1, JP-1 to MASTER, PW to POWER
Connections:
- removed net CS1: IC1.RCK, MASTER.4
- removed net N$3: D1.C, L1.1
- removed net N$5: IN.3, IN.4, OUT.3, OUT.4
- removed net N$6: IN.5, IN.6, OUT.5, OUT.6
- new net CS: IC1.RCK, IN.5, IN.6, MASTER.4, OUT.5, OUT.6
- new net VCC: C5.+, IC2.VIN, L1.2
- net +12V: now also D1.C, L1.1; no longer C5.+, IC2.IN, L1.2
- net +3V3: now also IC2.VOUT; no longer IC2.OUT
- net EXT_SERIAL: now also SLV.1
- net PA5: now also IN.3, IN.4, OUT.3, OUT.4
- net PA7: now also SLV.2
Other:
- moved on the sheet: C2, C4, C6
